File: Eagle/quad.sch (EAGLE design)
At the start: 20 parts

Commit message: Large board done
Connections:
- removed net N$26 (its old number): MODUL2.D6, USRIGHT.2
- removed net N$27: MODUL2.D7, USRIGHT.3
- removed net N$30: MODUL2.D8, USBACK.2
- new net N$2: MODUL2.D8, USLEFT.2
- new net N$28: MODUL2.D7, USLEFT.3
- new net N$32: MODUL2.D6, USBACK.3
- net N$22: now also MODUL2.D5, USBACK.2; no longer MODUL2.D4, USFRONT.2
- net N$23: now also MODUL2.D12/MISO, USRIGHT.3; no longer MODUL2.D5, USFRONT.3
- net N$24: now also MODUL2.D11/MOSI, USRIGHT.2; no longer MODUL2.D2, USLEFT.2
- net N$25: now also MODUL2.D10, USFRONT.2; no longer MODUL2.D3, USLEFT.3
- net N$29: now also USFRONT.3; no longer USBACK.3
Other:
- moved on the sheet: USBACK, USFRONT, USLEFT, USRIGHT
